Commit message: fixing urdf description frames for boris and tables

File: vito_description/robot/boris.urdf.xacro (robot description, xacro)
@@ -13,22 +13,23 @@
   <xacro:model_table name="table"
                     parent="vito_anchor"
-                    length="0.725"
-                    width="1.05"
+                    length="0.15"
+                    width="0.15"
                     height="0.910"
                     plate_thickness="0.05">
-    <origin xyz="-0.495 0.55 0" rpy="0 0 0"/>
+    <origin xyz="-0.075 0.075 0" rpy="0 0 0"/>
+    <!-- <origin xyz="0.495 0.55 0" rpy="0 0 0"/> -->
   </xacro:model_table>
   <!-- WORKBENCH -->
   <xacro:model_table name="workbench"
                     parent="vito_anchor"
-                    length="0.725"
-                    width="1.25"
-                    height="0.960"
-                    plate_thickness="0.1">
-  <origin xyz="-1.25 0.625 0.07" rpy="0 0 0"/>
+                    length="0.87"
+                    width="1.77"
+                    height="0.82"
+                    plate_thickness="0.05">
+  <origin xyz="0.1 0.885 -0.285" rpy="0 0 0"/>
   </xacro:model_table>
   <!-- TORSO -->
   <xacro:model_torso name="torso" parent="vito_anchor">
-    <origin xyz="0 0 0"/>
+    <origin xyz="0 0 0" rpy="0 0 ${M_PI}"/>
   </xacro:model_torso>
   <!-- LEFT ARM -->
@@ -46,9 +47,9 @@
   <!-- RIGHT SOFTHAND -->
   <xacro:soft_hand parent="right_arm_7_link" name="right_hand" left="false" withAdaptiveTransmission="true" useMimicTag="$(arg use_mimic_tag)">
-    <origin xyz="0 0 0" rpy="0 0 0"/>
+    <origin xyz="0 0 0" rpy="0 0 ${M_PI}"/>
   </xacro:soft_hand>
   <!-- HEAD -->
   <xacro:kit_head name="head" parent="vito_anchor">
-    <origin xyz="0.0 0.0 ${0.55 + 0.1}" rpy="0.0 0.0 3.141592"/>
+    <origin xyz="0.0 0.0 ${0.55 + 0.1}" rpy="0.0 0.0 0.0"/>
   </xacro:kit_head>
 </robot>

Commit message: asus description for left arm, and moveit update to ignore collisions

File: vito_description/robot/boris.urdf.xacro (robot description, xacro)
@@ -6,4 +6,5 @@
   <xacro:include filename="$(find vito_description)/model/table.urdf.xacro"/>
   <xacro:include filename="$(find vito_description)/model/materials.urdf"/>
+  <xacro:include filename="$(find vito_description)/robot/depth_sensor.urdf.xacro"/>
   <xacro:include filename="$(find lwr_description)/model/kuka_lwr.urdf.xacro"/>
   <xacro:include filename="$(find soft_hand_description)/model/soft_hand.urdf.xacro"/>
@@ -37,4 +38,8 @@
 		<origin xyz="0 0.12853 0.20722" rpy="0 ${-75 * M_PI / 180} ${-90 * M_PI / 180}"/>
   </xacro:kuka_lwr>
+  <!-- LEFT DEPTH SENSOR -->
+  <xacro:depth_sensor name="left_depth_sensor" parent="left_arm_7_link">
+		<origin xyz="0 0.15 0.10" rpy="0 0 0"/>
+  </xacro:depth_sensor>
   <!-- LEFT SOFTHAND -->
   <xacro:soft_hand parent="left_arm_7_link" name="left_hand" left="true" withAdaptiveTransmission="true" useMimicTag="$(arg use_mimic_tag)">

Commit message: added wall model to boris urdf.xacro, maybe still need to check is the parameter values are ok

File: vito_description/robot/boris.urdf.xacro (robot description, xacro)
@@ -5,4 +5,5 @@
   <xacro:include filename="$(find vito_description)/model/torso.urdf.xacro"/>
   <xacro:include filename="$(find vito_description)/model/table.urdf.xacro"/>
+  <xacro:include filename="$(find vito_description)/model/wall.urdf.xacro"/>
   <xacro:include filename="$(find vito_description)/model/materials.urdf"/>
   <xacro:include filename="$(find vito_description)/robot/depth_sensor.urdf.xacro"/>
@@ -30,4 +31,13 @@
   <origin xyz="0.1 0.885 -0.285" rpy="0 0 0"/>
   </xacro:model_table>
+  <!-- WALL -->
+  <xacro:model_wall name="wall"
+                    parent="vito_anchor"
+                    wall_x="0.5"
+                    wall_y="2.0"
+                    wall_z="2.0">
+    <origin xyz="-0.80 0 0" rpy="0 0 0"/>
+    <!-- <origin xyz="0.495 0.55 0" rpy="0 0 0"/> -->
+  </xacro:model_wall>
   <!-- TORSO -->
   <xacro:model_torso name="torso" parent="vito_anchor">

File: vito_description/robot/environment.urdf.xacro (robot description, xacro)
@@ -4,4 +4,5 @@
   <!-- MODELS -->
   <xacro:include filename="$(find vito_description)/model/table.urdf.xacro"/>
+  <xacro:include filename="$(find vito_description)/model/wall.urdf.xacro"/>
   <xacro:include filename="$(find vito_description)/model/materials.urdf"/>
   <!-- WORKBENCH -->

File: vito_description/robot/vito.urdf.xacro (robot description, xacro)
@@ -5,4 +5,5 @@
   <xacro:include filename="$(find vito_description)/model/torso.urdf.xacro"/>
   <xacro:include filename="$(find vito_description)/model/table.urdf.xacro"/>
+   <xacro:include filename="$(find vito_description)/model/wall.urdf.xacro"/>
   <xacro:include filename="$(find vito_description)/model/materials.urdf"/>
   <xacro:include filename="$(find lwr_description)/model/kuka_lwr.urdf.xacro"/>
@@ -28,4 +29,13 @@
   <origin xyz="-1.25 0.625 0.07" rpy="0 0 0"/>
   </xacro:model_table>
+  <!-- WALL -->
+  <xacro:model_wall name="wall"
+                    parent="vito_anchor"
+                    wall_x="0.5"
+                    wall_y="2.0"
+                    wall_z="2.0">
+    <origin xyz="-0.075 0.075 0" rpy="0 0 0"/>
+    <!-- <origin xyz="0.495 0.55 0" rpy="0 0 0"/> -->
+  </xacro:model_wall>
   <!-- TORSO -->
   <xacro:model_torso name="torso" parent="vito_anchor">

File: vito_description/robot/vito_calib.urdf.xacro (robot description, xacro)
@@ -3,4 +3,5 @@
        name="vito_calib">
   <xacro:include filename="$(find vito_description)/model/torso.urdf.xacro"/>
+  <xacro:include filename="$(find vito_description)/model/wall.urdf.xacro"/>
   <xacro:include filename="$(find vito_description)/model/table.urdf.xacro"/>
   <xacro:include filename="$(find vito_description)/model/materials.urdf"/>

File: vito_description/robot/vito_iliad.urdf.xacro (robot description, xacro)
@@ -4,4 +4,5 @@
   <!-- MODELS -->
   <xacro:include filename="$(find vito_description)/model/torso.urdf.xacro"/>
+  <xacro:include filename="$(find vito_description)/model/wall.urdf.xacro"/>
   <xacro:include filename="$(find vito_description)/model/table.urdf.xacro"/>
   <xacro:include filename="$(find vito_description)/model/velvet.urdf.xacro"/>

Commit message: functional depth sensors for the arm and external

File: vito_description/robot/boris.urdf.xacro (robot description, xacro)
@@ -50,5 +50,9 @@
   <!-- LEFT DEPTH SENSOR -->
   <xacro:depth_sensor name="left_depth_sensor" parent="left_arm_7_link">
-		<origin xyz="0 0.15 0.10" rpy="0 0 0"/>
+		<origin xyz="0 0.30 0.10" rpy="0 0 0"/>
+  </xacro:depth_sensor>
+  <!-- EXTERNAL DEPTH SENSOR -->
+  <xacro:depth_sensor name="external_depth_sensor" parent="vito_anchor">
+		<origin xyz="0.2 0.885 -0.0" rpy="0 ${30 * M_PI / 180} ${-90 * M_PI / 180}"/>
   </xacro:depth_sensor>
   <!-- LEFT SOFTHAND -->

File: vito_description/robot/depth_sensor.urdf.xacro (robot description, xacro)
@@ -25,4 +25,69 @@
       </collision>
     </link>
+  <!-- ASUS Xtion -->
+  <link name="${name}_camera_depth_frame"/>
+  <link name="${name}_camera_rgb_frame"/>
+  <link name="${name}_camera_depth_optical_frame"/>
+  <link name="${name}_camera_rgb_optical_frame"/>
+  <joint name="${name}_camera_depth_frame_joint" type="fixed" >
+    <origin rpy="0 0 0" xyz="0 0.045 0.02" />
+    <parent link="${name}_asus_link"/>
+    <child link="${name}_camera_depth_frame"/>
+  </joint>
+  <joint name="${name}_camera_rgb_frame_joint" type="fixed">
+    <origin rpy="0.0 0.0 0.0" xyz="0 0.02 0.02"/>
+    <parent link="${name}_asus_link"/>
+    <child link="${name}_camera_rgb_frame"/>
+  </joint>
+  <joint name="${name}_camera_depth_optical_frame_joint" type="fixed" >
+    <origin rpy="${-M_PI/2} 0 ${-M_PI/2}" xyz="0 0 0" />
+    <parent link="${name}_camera_depth_frame"/>
+    <child link="${name}_camera_depth_optical_frame"/>
+  </joint>
+  <joint name="${name}_camera_rgb_optical_frame_joint" type="fixed" >
+    <origin rpy="${-M_PI/2} 0 ${-M_PI/2}" xyz="0 0 0" />
+    <parent link="${name}_camera_rgb_frame"/>
+    <child link="${name}_camera_rgb_optical_frame"/>
+  </joint>
+  <gazebo reference="${name}_camera_depth_frame">
+    <sensor type="depth" name="${name}_camera_gazebo_sensor">
+      <always_on>true</always_on>
+      <update_rate>10.0</update_rate>
+      <camera>
+        <horizontal_fov>${57.0*M_PI/180.0}</horizontal_fov>
+        <image>
+          <format>B8G8R8</format>
+          <width>640</width>
+          <height>480</height>
+        </image>
+        <clip>
+          <near>0.01</near>
+          <far>5</far>
+        </clip>
+      </camera>
+      <plugin name="${name}_camera_link_controller" filename="libgazebo_ros_openni_kinect.so">
+        <alwaysOn>true</alwaysOn>
+        <updateRate>0</updateRate>
+        <cameraName>camera</cameraName>
+        <imageTopicName>${name}/camera/rgb/image_raw</imageTopicName>
+        <cameraInfoTopicName>${name}/camera/rgb/camera_info</cameraInfoTopicName>
+        <depthImageTopicName>${name}/camera/depth/image_raw</depthImageTopicName>
+        <depthImageCameraInfoTopicName>${name}/camera/depth/camera_info</depthImageCameraInfoTopicName>
+        <pointCloudTopicName>${name}/camera/depth_registered/points</pointCloudTopicName>
+        <frameName>${name}_camera_depth_optical_frame</frameName>
+        <pointCloudCutoff>0.05</pointCloudCutoff>
+        <distortionK1>0.0000000</distortionK1>
+        <distortionK2>0.0000000</distortionK2>
+        <distortionK3>0.0000000</distortionK3>
+        <distortionT1>0.0000000</distortionT1>
+        <distortionT2>0.0000000</distortionT2>
+        <CxPrime>0</CxPrime>
+        <Cx>0</Cx>
+        <Cy>0</Cy>
+        <focalLength>0</focalLength>
+        <hackBaseline>0</hackBaseline>
+      </plugin>
+    </sensor>
+    </gazebo>
     </xacro:macro>
 </robot>
