Commit message: updated transformations and fixed jittering table

File: boris_description/model/table.urdf.xacro (robot description, xacro)
@@ -9,5 +9,5 @@
 <xacro:property name="gr_to_Kg" value="0.001"/>
 <!-- not so negligible, otherwise simulation fails -->
-<xacro:property name="table_mass" value="${40000*gr_to_Kg}"/>
+<xacro:property name="table_mass" value="${500000*gr_to_Kg}"/>
 <xacro:property name="table_inertia">
     <origin xyz="0 0 0"/>
@@ -38,5 +38,5 @@
     </link>
     <gazebo reference="${name}_link">
-        <!-- <static>true</static> -->
+        <static>true</static>
     </gazebo>
 </xacro:macro>
@@ -78,5 +78,5 @@
     </xacro:table_leg>
     <gazebo reference="${name}_plate_link">
-        <!-- <static>true</static> -->
+        <static>true</static>
     </gazebo>
 </xacro:macro>

File: boris_description/robot/boris.urdf.xacro (robot description, xacro)
@@ -29,5 +29,5 @@
                     height="0.82"
                     plate_thickness="0.05">
-  <origin xyz="0.1 0.885 -0.285" rpy="0 0 0"/>
+  <origin xyz="0.1 0.885 -0.285" rpy="0 0 0"/> <!-- -0.285 -->
   </xacro:model_table>
   <!-- WALL -->
@@ -58,5 +58,5 @@
   <!-- LEFT SOFTHAND -->
   <xacro:soft_hand parent="left_arm_7_link" name="left_hand" left="true" withAdaptiveTransmission="true" useMimicTag="$(arg use_mimic_tag)">
-    <origin xyz="0 0 0" rpy="0 0 0"/>
+    <origin xyz="0 0 0.055" rpy="0 0 ${-135 * M_PI / 180}"/>
   </xacro:soft_hand>
   <!-- RIGHT ARM -->
@@ -64,11 +64,15 @@
 		<origin xyz="0 -0.12853 0.20722" rpy="0 ${75 * M_PI / 180} ${-90 * M_PI / 180}"/>
   </xacro:kuka_lwr>
+  <!-- RIGHT DEPTH SENSOR -->
+  <xacro:depth_sensor name="right_depth_sensor" parent="right_arm_7_link">
+		<origin xyz="0 0.30 0.10" rpy="0 0 0"/>
+  </xacro:depth_sensor>
   <!-- RIGHT SOFTHAND -->
   <xacro:soft_hand parent="right_arm_7_link" name="right_hand" left="false" withAdaptiveTransmission="true" useMimicTag="$(arg use_mimic_tag)">
-    <origin xyz="0 0 0" rpy="0 0 ${M_PI}"/>
+    <origin xyz="0 0 0.055" rpy="0 0 ${-135 * M_PI / 180}"/>
   </xacro:soft_hand>
   <!-- HEAD -->
   <xacro:kit_head name="head" parent="world">
-    <origin xyz="0.0 0.0 ${0.55 + 0.1}" rpy="0.0 0.0 0.0"/>
+    <origin xyz="0.0 0.0 0.58" rpy="0.0 0.0 0.0"/>
   </xacro:kit_head>
 </robot>
