Commit message: fixing readme

File: boris_description/robot/boris.urdf.xacro (robot description, xacro)
@@ -50,5 +50,5 @@
   <!-- LEFT DEPTH SENSOR -->
   <xacro:depth_sensor name="left_depth_sensor" parent="left_arm_7_link">
-		<origin xyz="0 0.30 0.10" rpy="0 0 0"/>
+		<origin xyz="0.09015027 0.06883422 0.07705509" rpy="3.10604 0.00301307 -0.829402"/>
   </xacro:depth_sensor>
   <!-- <pose_euler pitch="0.00301307" roll="3.10604" v1="0.429287" v2="0.327782" v3="-0.366929" yaw="0.829402"></pose_euler> -->
@@ -67,6 +67,7 @@
   <!-- RIGHT DEPTH SENSOR -->
   <xacro:depth_sensor name="right_depth_sensor" parent="right_arm_7_link">
-		<origin xyz="0 0.30 0.10" rpy="0 0 0"/>
+		<origin xyz="0.0633612 -0.05191389 0.05191389" rpy="-8.90385e-006 -0.0156339 -0.0116152"/>
   </xacro:depth_sensor>
+  <!-- <pose_euler pitch="-0.0156339" roll="-8.90385e-006" v1="0.30172" v2="-0.247209" v3="-0.349544" yaw="0.0116152"></pose_euler> -->
   <!-- RIGHT SOFTHAND -->
   <xacro:soft_hand parent="right_arm_7_link" name="right_hand" left="false" withAdaptiveTransmission="true" useMimicTag="$(arg use_mimic_tag)">

Commit message: approximately correct camera poses and collision fixes inj srdf

File: boris_description/robot/boris.urdf.xacro (robot description, xacro)
@@ -50,5 +50,5 @@
   <!-- LEFT DEPTH SENSOR -->
   <xacro:depth_sensor name="left_depth_sensor" parent="left_arm_7_link">
-		<origin xyz="0.09015027 0.06883422 0.07705509" rpy="3.10604 0.00301307 -0.829402"/>
+		<origin xyz="0.09015027 0.06883422 0.07705509" rpy="3.10604 0.0 0.00301307"/>
   </xacro:depth_sensor>
   <!-- <pose_euler pitch="0.00301307" roll="3.10604" v1="0.429287" v2="0.327782" v3="-0.366929" yaw="0.829402"></pose_euler> -->
@@ -67,5 +67,5 @@
   <!-- RIGHT DEPTH SENSOR -->
   <xacro:depth_sensor name="right_depth_sensor" parent="right_arm_7_link">
-		<origin xyz="0.0633612 -0.05191389 0.05191389" rpy="-8.90385e-006 -0.0156339 -0.0116152"/>
+		<origin xyz="-0.0633612 -0.05191389 0.05191389" rpy="${M_PI-8.90385e-006} 0.0156339 ${M_PI-0.0116152}"/>
   </xacro:depth_sensor>
   <!-- <pose_euler pitch="-0.0156339" roll="-8.90385e-006" v1="0.30172" v2="-0.247209" v3="-0.349544" yaw="0.0116152"></pose_euler> -->

Commit message: preparing for extrinsics calibration, done intrinsics and fixes to rviz, srdf, depth camera and adding scripts

File: boris_description/robot/boris.urdf.xacro (robot description, xacro)
@@ -49,12 +49,12 @@
   </xacro:kuka_lwr>
   <!-- LEFT DEPTH SENSOR -->
-  <xacro:depth_sensor name="left_depth_sensor" parent="left_arm_7_link">
+  <xacro:depth_sensor name="left" parent="left_arm_7_link">
 		<origin xyz="0.09015027 0.06883422 0.07705509" rpy="3.10604 0.0 0.00301307"/>
   </xacro:depth_sensor>
   <!-- <pose_euler pitch="0.00301307" roll="3.10604" v1="0.429287" v2="0.327782" v3="-0.366929" yaw="0.829402"></pose_euler> -->
   <!-- EXTERNAL DEPTH SENSOR -->
-  <xacro:depth_sensor name="external_depth_sensor" parent="world">
+  <!-- <xacro:depth_sensor name="external" parent="world">
 		<origin xyz="0.2 0.885 -0.0" rpy="0 ${30 * M_PI / 180} ${-90 * M_PI / 180}"/>
-  </xacro:depth_sensor>
+  </xacro:depth_sensor> -->
   <!-- LEFT SOFTHAND -->
   <xacro:soft_hand parent="left_arm_7_link" name="left_hand" left="false" withAdaptiveTransmission="true" useMimicTag="$(arg use_mimic_tag)">
@@ -66,5 +66,5 @@
   </xacro:kuka_lwr>
   <!-- RIGHT DEPTH SENSOR -->
-  <xacro:depth_sensor name="right_depth_sensor" parent="right_arm_7_link">
+  <xacro:depth_sensor name="right" parent="right_arm_7_link">
 		<origin xyz="-0.0633612 -0.05191389 0.05191389" rpy="${M_PI-8.90385e-006} 0.0156339 ${M_PI-0.0116152}"/>
   </xacro:depth_sensor>

File: boris_description/robot/depth_sensor.urdf.xacro (robot description, xacro)
@@ -5,7 +5,7 @@
       <xacro:insert_block name="origin"/>
       <parent link="${parent}"/>
-      <child link="${name}_asus_link"/>
+      <child link="${name}_camera_link"/>
     </joint>
-    <link name="${name}_asus_link">
+    <link name="${name}_camera_link">
       <inertial>
         <xacro:insert_block name="negligible_inertia"/>
@@ -32,10 +32,10 @@
   <joint name="${name}_camera_depth_frame_joint" type="fixed" >
     <origin rpy="0 0 0" xyz="0 0.045 0.02" />
-    <parent link="${name}_asus_link"/>
+    <parent link="${name}_camera_link"/>
     <child link="${name}_camera_depth_frame"/>
   </joint>
   <joint name="${name}_camera_rgb_frame_joint" type="fixed">
     <origin rpy="0.0 0.0 0.0" xyz="0 0.02 0.02"/>
-    <parent link="${name}_asus_link"/>
+    <parent link="${name}_camera_link"/>
     <child link="${name}_camera_rgb_frame"/>
   </joint>

Commit message: kinetic fixes and left camera calibration

File: boris_description/robot/boris.urdf.xacro (robot description, xacro)
@@ -28,6 +28,6 @@
                     width="1.77"
                     height="0.82"
-                    plate_thickness="0.05">
-  <origin xyz="0.1 0.885 -0.285" rpy="0 0 0"/> <!-- -0.285 -->
+                    plate_thickness="0.025">
+  <origin xyz="0.1 0.885 -0.33" rpy="0 0 0"/> <!-- -0.285 -->
   </xacro:model_table>
   <!-- WALL -->
@@ -49,8 +49,12 @@
   </xacro:kuka_lwr>
   <!-- LEFT DEPTH SENSOR -->
+  <!-- [0.1034412  0.00049388 0.08871709]
+[-3.12590633 -0.00839937 -0.06241149] -->
   <xacro:depth_sensor name="left" parent="left_arm_7_link">
-		<origin xyz="0.09015027 0.06883422 0.07705509" rpy="3.10604 0.0 0.00301307"/>
+		<origin xyz="0.09221578 0.00125629 0.08367657" rpy="-3.12900506 -0.01153159 -0.06345897"/> <!--3.10604 0.0 0.00301307-->
   </xacro:depth_sensor>
+  <!--0.09221578 0.00125629 0.08367657-->
   <!-- <pose_euler pitch="0.00301307" roll="3.10604" v1="0.429287" v2="0.327782" v3="-0.366929" yaw="0.829402"></pose_euler> -->
+<!-- <origin xyz="0.09015027 0.06883422 0.07705509" rpy="3.10604 0.0 0.00301307"/> -->
   <!-- EXTERNAL DEPTH SENSOR -->
   <!-- <xacro:depth_sensor name="external" parent="world">
@@ -59,5 +63,5 @@
   <!-- LEFT SOFTHAND -->
   <xacro:soft_hand parent="left_arm_7_link" name="left_hand" left="false" withAdaptiveTransmission="true" useMimicTag="$(arg use_mimic_tag)">
-    <origin xyz="0 0 0.055" rpy="0 0 ${-135 * M_PI / 180}"/>
+    <origin xyz="0 0 0.072" rpy="0 0 ${-135 * M_PI / 180}"/>
   </xacro:soft_hand>
   <!-- RIGHT ARM -->
@@ -72,5 +76,5 @@
   <!-- RIGHT SOFTHAND -->
   <xacro:soft_hand parent="right_arm_7_link" name="right_hand" left="false" withAdaptiveTransmission="true" useMimicTag="$(arg use_mimic_tag)">
-    <origin xyz="0 0 0.055" rpy="0 0 ${-135 * M_PI / 180}"/>
+    <origin xyz="0 0 0.072" rpy="0 0 ${-135 * M_PI / 180}"/><!--055-->
   </xacro:soft_hand>
   <!-- HEAD -->

File: boris_description/robot/depth_sensor.urdf.xacro (robot description, xacro)
@@ -12,5 +12,5 @@
       </inertial>
       <visual>
-        <origin xyz="0 0 0" rpy="0 0 0"/>
+        <origin xyz="0 0 0" rpy="0 0 0.0"/>
         <geometry>
           <mesh filename="package://boris_description/meshes/asus_xtion_body.stl"/>
@@ -31,10 +31,10 @@
   <link name="${name}_camera_rgb_optical_frame"/>
   <joint name="${name}_camera_depth_frame_joint" type="fixed" >
-    <origin rpy="0 0 0" xyz="0 0.045 0.02" />
+    <origin rpy="0 0 0" xyz="0 0.045 0.0" />
     <parent link="${name}_camera_link"/>
     <child link="${name}_camera_depth_frame"/>
   </joint>
   <joint name="${name}_camera_rgb_frame_joint" type="fixed">
-    <origin rpy="0.0 0.0 0.0" xyz="0 0.02 0.02"/>
+    <origin rpy="0.0 0.0 0.0" xyz="0 0.022 0.0"/>
     <parent link="${name}_camera_link"/>
     <child link="${name}_camera_rgb_frame"/>

Commit message: right arm calibration

File: boris_description/robot/boris.urdf.xacro (robot description, xacro)
@@ -71,5 +71,5 @@
   <!-- RIGHT DEPTH SENSOR -->
   <xacro:depth_sensor name="right" parent="right_arm_7_link">
-		<origin xyz="-0.0633612 -0.05191389 0.05191389" rpy="${M_PI-8.90385e-006} 0.0156339 ${M_PI-0.0116152}"/>
+		<origin xyz="-0.07053522  0.00938331  0.07951935" rpy="0.10361832 -0.0499392  -2.99893557"/>
   </xacro:depth_sensor>
   <!-- <pose_euler pitch="-0.0156339" roll="-8.90385e-006" v1="0.30172" v2="-0.247209" v3="-0.349544" yaw="0.0116152"></pose_euler> -->

File: boris_description/robot/depth_sensor.urdf.xacro (robot description, xacro)
@@ -31,5 +31,5 @@
   <link name="${name}_camera_rgb_optical_frame"/>
   <joint name="${name}_camera_depth_frame_joint" type="fixed" >
-    <origin rpy="0 0 0" xyz="0 0.045 0.0" />
+    <origin rpy="0 0 0" xyz="0 0.049 0.0" />
     <parent link="${name}_camera_link"/>
     <child link="${name}_camera_depth_frame"/>

Commit message: calibrated bors

File: boris_description/robot/boris.urdf.xacro (robot description, xacro)
@@ -49,16 +49,7 @@
   </xacro:kuka_lwr>
   <!-- LEFT DEPTH SENSOR -->
-  <!-- [0.1034412  0.00049388 0.08871709]
-[-3.12590633 -0.00839937 -0.06241149] -->
   <xacro:depth_sensor name="left" parent="left_arm_7_link">
-		<origin xyz="0.09221578 0.00125629 0.08367657" rpy="-3.12900506 -0.01153159 -0.06345897"/> <!--3.10604 0.0 0.00301307-->
+		<origin xyz="0.08962811 -0.00032633 0.08260346" rpy="-3.1290897546768672 -0.06293262669010466 -0.007904165374966"/>
   </xacro:depth_sensor>
-  <!--0.09221578 0.00125629 0.08367657-->
-  <!-- <pose_euler pitch="0.00301307" roll="3.10604" v1="0.429287" v2="0.327782" v3="-0.366929" yaw="0.829402"></pose_euler> -->
-<!-- <origin xyz="0.09015027 0.06883422 0.07705509" rpy="3.10604 0.0 0.00301307"/> -->
-  <!-- EXTERNAL DEPTH SENSOR -->
-  <!-- <xacro:depth_sensor name="external" parent="world">
-		<origin xyz="0.2 0.885 -0.0" rpy="0 ${30 * M_PI / 180} ${-90 * M_PI / 180}"/>
-  </xacro:depth_sensor> -->
   <!-- LEFT SOFTHAND -->
   <xacro:soft_hand parent="left_arm_7_link" name="left_hand" left="false" withAdaptiveTransmission="true" useMimicTag="$(arg use_mimic_tag)">
@@ -68,10 +59,9 @@
   <xacro:kuka_lwr name="right_arm" parent="world">
 		<origin xyz="0 -0.12853 0.20722" rpy="0 ${75 * M_PI / 180} ${-90 * M_PI / 180}"/>
-  </xacro:kuka_lwr>
+  </xacro:kuka_lwr><!-- 0 -0.12853 0.20722-->
   <!-- RIGHT DEPTH SENSOR -->
   <xacro:depth_sensor name="right" parent="right_arm_7_link">
-		<origin xyz="-0.07053522  0.00938331  0.07951935" rpy="0.10361832 -0.0499392  -2.99893557"/>
+		<origin xyz="-0.0751738 -0.00186555 0.08051474" rpy="3.131270940071478 -0.08173348350733739 -3.1183375574826124"/>
   </xacro:depth_sensor>
-  <!-- <pose_euler pitch="-0.0156339" roll="-8.90385e-006" v1="0.30172" v2="-0.247209" v3="-0.349544" yaw="0.0116152"></pose_euler> -->
   <!-- RIGHT SOFTHAND -->
   <xacro:soft_hand parent="right_arm_7_link" name="right_hand" left="false" withAdaptiveTransmission="true" useMimicTag="$(arg use_mimic_tag)">
@@ -80,5 +70,5 @@
   <!-- HEAD -->
   <xacro:kit_head name="head" parent="world">
-    <origin xyz="0.0 0.0 0.58" rpy="0.0 0.0 0.0"/>
+    <origin xyz="0.0 0.0 0.61" rpy="0.0 0.0 0.0"/> <!-- 0.58 -->
   </xacro:kit_head>
 </robot>

File: boris_description/robot/depth_sensor.urdf.xacro (robot description, xacro)
@@ -31,5 +31,5 @@
   <link name="${name}_camera_rgb_optical_frame"/>
   <joint name="${name}_camera_depth_frame_joint" type="fixed" >
-    <origin rpy="0 0 0" xyz="0 0.049 0.0" />
+    <origin rpy="0 0 0" xyz="0 0.047 0.0" />
     <parent link="${name}_camera_link"/>
     <child link="${name}_camera_depth_frame"/>

Commit message: moveit example

File: boris_description/robot/boris.urdf.xacro (robot description, xacro)
@@ -70,5 +70,6 @@
   <!-- HEAD -->
   <xacro:kit_head name="head" parent="world">
-    <origin xyz="0.0 0.0 0.61" rpy="0.0 0.0 0.0"/> <!-- 0.58 -->
+    <origin xyz="0.0 0.0 0.61" rpy="0.0 0.0 0.0"/>
   </xacro:kit_head>
+  <!-- 0.58 -->
 </robot>

Commit message: adding force torque link, calibrated f/t tools and mock_imu

File: boris_description/robot/boris.urdf.xacro (robot description, xacro)
@@ -37,5 +37,5 @@
                     wall_y="2.0"
                     wall_z="2.0">
-    <origin xyz="-0.80 0 0" rpy="0 0 0"/>
+    <origin xyz="-0.40 0 0" rpy="0 0 0"/>
     <!-- <origin xyz="0.495 0.55 0" rpy="0 0 0"/> -->
   </xacro:model_wall>
@@ -53,6 +53,12 @@
   </xacro:depth_sensor>
   <!-- LEFT SOFTHAND -->
-  <xacro:soft_hand parent="left_arm_7_link" name="left_hand" left="false" withAdaptiveTransmission="false" useMimicTag="$(arg use_mimic_tag)">
-    <origin xyz="0 0 0.072" rpy="0 0 ${-135 * M_PI / 180}"/>
+  <link name="left_ft_sensor" />
+  <joint name="left_ft_sensor_joint" type="fixed" >
+    <origin rpy="0 0 ${45 * M_PI / 180}" xyz="0 0.0 0.0" />
+    <parent link="left_arm_7_link"/>
+    <child link="left_ft_sensor"/>
+  </joint>
+  <xacro:soft_hand parent="left_ft_sensor" name="left_hand" left="false" withAdaptiveTransmission="false" useMimicTag="$(arg use_mimic_tag)">
+    <origin xyz="0 0 0.072" rpy="0 0 ${-180 * M_PI / 180}"/>
   </xacro:soft_hand>
   <!-- RIGHT ARM -->

Commit message: removing table temporarily

File: boris_description/robot/boris.urdf.xacro (robot description, xacro)
@@ -23,5 +23,5 @@
   </xacro:model_table>
   <!-- WORKBENCH -->
-  <xacro:model_table name="workbench"
+  <!-- <xacro:model_table name="workbench"
                     parent="world"
                     length="0.87"
@@ -29,6 +29,7 @@
                     height="0.82"
                     plate_thickness="0.025">
-  <origin xyz="0.1 0.885 -0.33" rpy="0 0 0"/> <!-- -0.285 -->
-  </xacro:model_table>
+  <origin xyz="0.1 0.885 -0.33" rpy="0 0 0"/>
+  </xacro:model_table> -->
+   <!-- -0.285 -->
   <!-- WALL -->
   <xacro:model_wall name="wall"

Commit message: adding box to product cable socket on wrist

File: boris_description/robot/boris.urdf.xacro (robot description, xacro)
@@ -53,4 +53,31 @@
 		<origin xyz="0.08962811 -0.00032633 0.08260346" rpy="-3.1290897546768672 -0.06293262669010466 -0.007904165374966"/>
   </xacro:depth_sensor>
+  <link name="left_cable_guards">
+    <inertial>
+      <origin xyz="0.0 0.0 0.0" />
+      <mass value="0.1" />
+      <inertia  ixx="1" ixy="0.0"  ixz="0.0"  iyy="1"  iyz="0.0"  izz="1" />
+    </inertial>
+    <!-- real size 7.5 11.5 22.5 -->
+    <visual>
+      <origin rpy="0 0 0"  xyz="0.0 0.0 0.0"/>
+      <geometry>
+        <box size="0.09 0.20 0.05" />
+      </geometry>
+      <material name="Boris/Silver"/>
+    </visual>
+    <collision>
+        <origin rpy="0 0 0"  xyz="0.0 0.0 0.0"/>
+       <box size="0.09 0.20 0.05" />
+      <geometry>
+         <box size="0.09 0.20 0.05" />
+      </geometry>
+    </collision>
+  </link>
+  <joint name="left_cable_guards_joint" type="fixed" >
+    <origin rpy="0 0 0" xyz="0 0.035 0.04" />
+    <parent link="left_arm_7_link"/>
+    <child link="left_cable_guards"/>
+  </joint>
   <!-- LEFT SOFTHAND -->
   <link name="left_ft_sensor" />

Commit message: box protecting the cables adjustment

File: boris_description/robot/boris.urdf.xacro (robot description, xacro)
@@ -76,5 +76,5 @@
   </link>
   <joint name="left_cable_guards_joint" type="fixed" >
-    <origin rpy="0 0 0" xyz="0 0.035 0.04" />
+    <origin rpy="0 0 0" xyz="0 -0.035 0.04" />
     <parent link="left_arm_7_link"/>
     <child link="left_cable_guards"/>

Commit message: setting up final experiments

File: boris_description/robot/boris.urdf.xacro (robot description, xacro)
@@ -23,5 +23,5 @@
   </xacro:model_table>
   <!-- WORKBENCH -->
-  <!-- <xacro:model_table name="workbench"
+  <xacro:model_table name="workbench"
                     parent="world"
                     length="0.87"
@@ -30,5 +30,5 @@
                     plate_thickness="0.025">
   <origin xyz="0.1 0.885 -0.33" rpy="0 0 0"/>
-  </xacro:model_table> -->
+  </xacro:model_table>
    <!-- -0.285 -->
   <!-- WALL -->

File: boris_tools/models/object.urdf (robot description, URDF)
Before this commit: robot object, 1 links, 0 joints
Links:
- link object: mass 0.1 -> 0.5
